File: Arm_PCB/Arm_PCB.kicad_pcb (KiCad board)
At the start: 2 copper layers, 123 parts, among them J1 Conn_02x04_Counter_Clockwise, J10 Conn_02x02_Counter_Clockwise, J11 Conn_02x04_Counter_Clockwise, J12 Screw_Terminal_01x02, J13 Screw_Terminal_01x02, J14 Screw_Terminal_01x02, J15 Screw_Terminal_01x02, J16 Screw_Terminal_01x02, J17 Screw_Terminal_01x02, J18 Screw_Terminal_01x02, J19 Conn_02x03_Counter_Clockwise, J2 Conn_02x04_Counter_Clockwise, J20 Conn_02x03_Counter_Clockwise, J3 Conn_02x04_Counter_Clockwise, J4 Conn_02x04_Counter_Clockwise, J5 Conn_02x03_Counter_Clockwise, J6 Conn_02x07_Counter_Clockwise, J7 Conn_02x03_Counter_Clockwise, J8 Conn_02x02_Counter_Clockwise, J9 Conn_02x04_Counter_Clockwise, SW1 SW_Push, SW2 SW_Push, SW3 SW_Push, SW4 SW_Push, U1 TB6560_Board, U10 TB6560_Board, U11 INA219AxDCN, U12 TB6560_Board, U13 INA219AxDCN, U14 TB6560_Board, U15 INA219AxDCN, U16 TB6560_Board, U2 INA219AxDCN, U3 INA219AxDCN, U4 INA219AxDCN, U5 TB6560_Board, U6 INA219AxDCN, U7 TB6560_Board, U8 INA219AxDCN, U9 INA219AxDCN

Commit message: Create good footprint for TB6560 driver
Parts:
- added J21: Screw_Terminal_01x02, TerminalBlock:TerminalBlock_bornier-2_P5.08mm, F.Cu at (266.7, 141.3)
- added J22: Screw_Terminal_01x02, TerminalBlock:TerminalBlock_bornier-2_P5.08mm, F.Cu at (266.7, 150.3)
- added J23: Screw_Terminal_01x02, TerminalBlock:TerminalBlock_bornier-2_P5.08mm, F.Cu at (266.7, 159.4)
- added J24: Screw_Terminal_01x02, TerminalBlock:TerminalBlock_bornier-2_P5.08mm, F.Cu at (266.7, 168.4)
- added J25: Screw_Terminal_01x02, TerminalBlock:TerminalBlock_bornier-2_P5.08mm, F.Cu at (266.7, 177.5)
- added J26: Screw_Terminal_01x02, TerminalBlock:TerminalBlock_bornier-2_P5.08mm, F.Cu at (266.7, 186.5)
- added J27: Screw_Terminal_01x02, TerminalBlock:TerminalBlock_bornier-2_P5.08mm, F.Cu at (266.7, 195.6)
- moved XA1 92.7 mm to (389.9, 175.3)
- moved XA2 69.1 mm to (344.2, 195.6)
- moved D6 14.9 mm to (183.3, 161.5)
- moved J12 14.9 mm to (204.2, 218.1)
- moved J19 14.9 mm to (233.1, 197.1)
- moved J9 14.9 mm to (133.2, 201.5)
- moved R1 14.9 mm to (209.9, 183.1)
- moved R15 14.9 mm to (221.8, 183.1)
- moved R16 14.9 mm to (221.8, 186.3)
- moved R19 14.9 mm to (221.8, 196.2)
- moved R2 14.9 mm to (209.9, 186.3)
- moved R44 14.9 mm to (177.3, 144.5)
- moved R47 14.9 mm to (177.3, 154.3)
- moved R5 14.9 mm to (209.9, 196.2)
- moved R50 14.9 mm to (177.3, 164.2)
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
Commit message: Grouped parts in the PCB sketch to begin routing
Parts:
- moved JP5 302.4 mm to (386.1, 226.1)
- moved J11 243.3 mm to (383.5, 211.7)
- moved J8 229.2 mm to (358.1, 226.9)
- moved J9 225.2 mm to (358.1, 211.7)
- moved J27 215.7 mm to (61.0, 260.4)
- moved J26 214.0 mm to (61.0, 245.5)
- moved J25 212.5 mm to (61.0, 230.7)
- moved J23 211.7 mm to (81.3, 261.6)
- moved J24 211.1 mm to (61.0, 215.9)
- moved J22 209.0 mm to (81.3, 246.8)
- moved J21 206.4 mm to (81.3, 232.0)
- moved U11 192.1 mm to (298.6, 250.5)
- moved J1 180.9 mm to (269.2, 127.0)
- moved J2 180.9 mm to (276.4, 127.0)
- moved J5 180.9 mm to (262.0, 127.0)
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
Commit message: Continue layout, pick some components
Parts:
- added J12: Screw_Terminal_01x02, TerminalBlock:TerminalBlock_bornier-2_P5.08mm, F.Cu at (56.5, 147.3)
- added R51: 3.3k, Resistor_SMD:R_1206_3216Metric_Pad1.30x1.75mm_HandSolder, F.Cu at (179.4, 144.8)
- added R52: 3.3k, Resistor_SMD:R_1206_3216Metric_Pad1.30x1.75mm_HandSolder, F.Cu at (179.4, 141.0)
- BZ1: footprint Buzzer_Beeper:Buzzer_12x9.5RM7.6 -> Buzzer_Beeper:Buzzer_15x7.5RM7.6
- C1, C2, C3, C4, C5, C6, C7, C8, C9: value C -> 0.1u
- R1, R10, R11, R12, R19, R2, R20, R25, R3: value R -> 2m
- U11, U13, U15, U2, U3, U4, U6, U8, U9: footprint Package_TO_SOT_SMD:SOT-23-8 -> Package_SO:SOIC-8_3.9x4.9mm_P1.27mm
- moved J27 391.2 mm to (388.0, 45.7), turned to 180 degrees
- moved J26 340.9 mm to (337.2, 45.7), turned to 180 degrees
- moved R34 282.0 mm to (354.7, 58.4), turned to 180 degrees
- moved J24 281.4 mm to (285.1, 45.7), turned to 180 degrees
- moved D7 280.8 mm to (344.6, 45.7), turned to 180 degrees
- moved R9 280.5 mm to (67.0, 117.8)
- moved C2 280.5 mm to (50.2, 117.8)
- moved R3 280.5 mm to (50.2, 112.7)
- moved R8 280.5 mm to (67.0, 112.7)
- moved U4 280.5 mm to (59.0, 116.2)
- moved J25 253.5 mm to (234.3, 45.7), turned to 180 degrees
- moved D6 246.4 mm to (293.8, 45.7), turned to 180 degrees
- moved R33 243.4 mm to (301.3, 58.4), turned to 180 degrees
- moved J23 238.9 mm to (183.5, 45.7), turned to 180 degrees
- moved J11 220.8 mm to (165.7, 175.3), turned to 90 degrees
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Connections:
- XA2 pad A0: Net-(J9-Pin_7) -> Net-(J9-Pin_1)
- XA2 pad A1: Net-(J9-Pin_5) -> Net-(J9-Pin_3)
- XA2 pad A2: Net-(J9-Pin_3) -> Net-(J9-Pin_5)
- XA2 pad A3: Net-(J9-Pin_1) -> Net-(J9-Pin_7)
Other:
- board text added: "A0 A1 A2 A3"
- board text added: "ADC Mega"
- board text added: "ADC Nano"
- board text added: "D0 D1"
- board text added: "D0 D1 19 18"
- board text added: "D11 D12 D13"
- board text added: "D4 D5 D6 D7"
- board text added: "Dir Stp En"
- board text added: "GPIO Mega"
- board text added: "GPIO Nano"
- board text added: "GPIO/UART Mega"
- board text added: "M0 Debug"
- board text added: "RX TX"
- board text added: "S V G"
- board text added: "SCL"
- board text added: "SDA"
- board text added: "Servo 1"
- board text added: "Servo 2"
- board text added: "UART Nano"

Commit message: Footprint updates with new TB6600
Parts:
- U1, U16: footprint Arm_Footprints:TB6560_Breakout -> Arm_Footprints:TB6600_Breakout
- moved R28 52.8 mm to (100.0, 55.9)
- moved C2 50.6 mm to (100.5, 112.7)
- moved R3 50.6 mm to (100.5, 107.6)
- moved R8 50.6 mm to (117.3, 107.6)
- moved R9 50.6 mm to (117.3, 112.7)
- moved U4 50.6 mm to (109.3, 111.1)
- moved R50 40.3 mm to (244.4, 182.9)
- moved D13 40.3 mm to (252.5, 182.9)
- moved J27 40.0 mm to (348.0, 45.7)
- moved D1 38.8 mm to (77.3, 55.9)
- moved D2 36.4 mm to (127.0, 46.8), turned to 90 degrees
- moved R34 33.8 mm to (321.0, 55.9)
- moved R29 22.4 mm to (120.4, 55.9)
- moved U1 20.7 mm to (78.7, 91.4)
- moved U16 17.5 mm to (347.2, 88.9), turned to 180 degrees
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Other:
- board text added: "Spotlight"

Commit message: Update layout
Parts:
- removed the J12 at (53.3, 167.6)
- removed R13, R14, R15, R16, R17, R18, R21, R22, R23, R24, R26, R27, R4, R5, R6, R7, R8, R9: 10K, Resistor_SMD:R_1206_3216Metric_Pad1.30x1.75mm_HandSolder
- moved U13 38.9 mm to (325.1, 111.1)
- moved R20 38.4 mm to (317.5, 110.2), turned to -90 degrees
- moved D2 36.8 mm to (90.2, 46.8)
- moved C8 32.3 mm to (323.6, 116.8)
- moved C4 17.4 mm to (117.8, 119.4)
- moved U8 12.2 mm to (119.3, 113.7)
- moved R11 12.0 mm to (111.8, 112.8), turned to -90 degrees
- moved U4 10.5 mm to (99.1, 113.7)
- moved R3 10.4 mm to (91.4, 112.8), turned to -90 degrees
- moved J21 8.89 mm to (82.5, 45.7)
- moved C1 8.82 mm to (261.6, 119.4)
- moved U9 8.03 mm to (305.4, 111.1)
- moved C9 7.91 mm to (209.3, 119.4)
- moved R12 7.85 mm to (297.6, 110.2), turned to -90 degrees
- moved C3 7.75 mm to (140.7, 162.6)
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Connections:
- U11 pad 7: Net-(U11-A0) -> SDA
- U11 pad 8: Net-(U11-A1) -> GND
- U13 pad 7: Net-(U13-A0) -> SDA
- U13 pad 8: Net-(U13-A1) -> +5V
- U15 pad 7: Net-(U15-A0) -> SCL
- U15 pad 8: Net-(U15-A1) -> GND
- U2 pad 7: Net-(U2-A0) -> SCL
- U2 pad 8: Net-(U2-A1) -> +5V
- U3 pad 7: Net-(U3-A0) -> GND
- U3 pad 8: Net-(U3-A1) -> +5V
- U4 pad 7: Net-(U4-A0) -> GND
- U4 pad 8: Net-(U4-A1) -> GND
- U6 pad 7: Net-(U6-A0) -> GND
- U6 pad 8: Net-(U6-A1) -> SDA
- U8 pad 7: Net-(U8-A0) -> +5V
- U8 pad 8: Net-(U8-A1) -> GND
- U9 pad 7: Net-(U9-A0) -> +5V
- U9 pad 8: Net-(U9-A1) -> +5V
Other:
- board outline added: 332.7 x 149.9 mm
- board text added: "24V GND"
- board text added: "3V3"
- board text added: "3V3 GND"
- board text added: "5V"
- board text added: "5V GND"
- board text added: "Designed by Parker and Rolston"
- board text added: "GND"
- board text added: "GP LEDs and Buttons"
- board text added: "If nothing else, this darn board will beep."
- board text added: "Power: 24V"
- board text added: "Power: 3V3"
- board text added: "Power: 5V"
- board text added: "Rev 1.0 - the only rev ;)"
- board text added: "SSRT 2023 Robot Arm Control Board"

Commit message: Start routing
Routing:
- net +24V: track 0.00 -> 436.2 mm
- net +5V: track 0.00 -> 293.3 mm
- net M0_STEP: track 0.00 -> 261.9 mm, vias 0 -> 2
- net M0_DIR: track 0.00 -> 244.1 mm, vias 0 -> 1
- net M0_EN: track 0.00 -> 236.6 mm, vias 0 -> 2
- net MPOWER2: track 0.00 -> 116.5 mm, vias 0 -> 11
- net MPOWER3: track 0.00 -> 105.8 mm, vias 0 -> 9
- net MPOWER4: track 0.00 -> 100.2 mm, vias 0 -> 9
- net MPOWER5: track 0.00 -> 97.9 mm, vias 0 -> 9
- net MPOWER1: track 0.00 -> 94.2 mm, vias 0 -> 8
- net MPOWER0: track 0.00 -> 85.4 mm, vias 0 -> 9
- net MPOWER6: track 0.00 -> 52.5 mm, vias 0 -> 9
- added copper zone on F.Cu, net GND

Commit message: Route more
Parts:
- removed D1, D2, D3, D4, D5, D6, D7: LED, LED_SMD:LED_1206_3216Metric_Pad1.42x1.75mm_HandSolder
- removed R28, R29, R30, R31, R32, R33, R34: R, Resistor_SMD:R_1206_3216Metric_Pad1.30x1.75mm_HandSolder
- moved JP3 15.5 mm to (203.8, 170.2), turned to 90 degrees
- moved JP4 4.44 mm to (203.8, 174.6)
- moved R1 0.63 mm to (135.3, 155.9)
Connections:
- net Net-(J19-Pin_3) renamed /MotorDrivers/S_POWER_1
- net Net-(J20-Pin_3) renamed /MotorDrivers/S_POWER_2
Routing:
- net +5V: track 293.3 -> 594.9 mm, vias 0 -> 5
- net Net-(JP3-A): track 0.00 -> 216.2 mm, vias 0 -> 3
- net M6_EN: track 0.00 -> 214.8 mm, vias 0 -> 2
- net M6_DIR: track 0.00 -> 202.1 mm, vias 0 -> 2
- net M2_EN: track 0.00 -> 197.8 mm, vias 0 -> 2
- net M1_EN: track 0.00 -> 189.6 mm, vias 0 -> 1
- net M6_STEP: track 0.00 -> 186.1 mm, vias 0 -> 2
- net Net-(JP4-A): track 0.00 -> 185.6 mm, vias 0 -> 3
- net M2_DIR: track 0.00 -> 183.5 mm, vias 0 -> 2
- net M1_DIR: track 0.00 -> 181.2 mm, vias 0 -> 1
- net M1_STEP: track 0.00 -> 175.2 mm, vias 0 -> 1
- net Net-(JP4-B): track 0.00 -> 165.2 mm, vias 0 -> 3
- net BUZZER0: track 0.00 -> 155.7 mm, vias 0 -> 2
- net M2_STEP: track 0.00 -> 153.2 mm, vias 0 -> 2
- net SPOTLIGHT0: track 0.00 -> 135.7 mm, vias 0 -> 2
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Other:
- board text added: "1-2 for Mega"
- board text added: "I2C uC"
