File: Arm_PCB/Arm_PCB.kicad_pcb (KiCad board)
At the start: 2 copper layers, 332.7 x 149.9 mm, 100 parts, among them J1 Conn_02x04_Counter_Clockwise, J10 Conn_02x02_Counter_Clockwise, J11 Conn_02x04_Counter_Clockwise, J12 Screw_Terminal_01x02, J13 Screw_Terminal_01x02, J14 Screw_Terminal_01x02, J15 Screw_Terminal_01x02, J16 Screw_Terminal_01x02, J17 Screw_Terminal_01x02, J18 Screw_Terminal_01x02, J19 Conn_02x03_Counter_Clockwise, J2 Conn_02x04_Counter_Clockwise, J20 Conn_02x03_Counter_Clockwise, J21 Screw_Terminal_01x02, J22 Screw_Terminal_01x02, J23 Screw_Terminal_01x02, J24 Screw_Terminal_01x02, J25 Screw_Terminal_01x02, J26 Screw_Terminal_01x02, J27 Screw_Terminal_01x02, J3 Conn_02x04_Counter_Clockwise, J4 Conn_02x04_Counter_Clockwise, J5 Conn_02x03_Counter_Clockwise, J6 Conn_02x07_Counter_Clockwise, J7 Conn_02x03_Counter_Clockwise, J8 Conn_02x02_Counter_Clockwise, J9 Conn_02x04_Counter_Clockwise, SW1 SW_Push, SW2 SW_Push, SW3 SW_Push, SW4 SW_Push, U1 TB6560_Board, U10 TB6560_Board, U11 INA219AxDCN, U12 TB6560_Board, U13 INA219AxDCN, U14 TB6560_Board, U15 INA219AxDCN, U16 TB6560_Board, U2 INA219AxDCN, U3 INA219AxDCN, U4 INA219AxDCN, U5 TB6560_Board, U6 INA219AxDCN, U7 TB6560_Board, U8 INA219AxDCN, U9 INA219AxDCN

Commit message: Route more, move uC to middle
Parts:
- moved R51 113.7 mm to (292.5, 145.4)
- moved R52 113.7 mm to (292.5, 141.6)
- moved J10 113.7 mm to (299.7, 142.9)
- moved JP1 112.5 mm to (103.5, 183.5), turned to 90 degrees
- moved J1 111.4 mm to (281.3, 155.6)
- moved J11 111.4 mm to (281.3, 165.7)
- moved J2 111.4 mm to (297.8, 155.6)
- moved J9 111.4 mm to (297.8, 165.7)
- moved XA2 110.1 mm to (264.8, 163.2)
- moved XA1 108.0 mm to (268.0, 191.1)
- moved JP2 101.0 mm to (112.4, 183.5), turned to 90 degrees
- moved D10 100.5 mm to (333.5, 158.4)
- moved D11 100.5 mm to (333.5, 163.5)
- moved D12 100.5 mm to (333.5, 168.6)
- moved D8 100.5 mm to (333.5, 147.6)
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Routing:
- net LIMIT6: track 5.08 -> 391.0 mm, vias 0 -> 11
- net LIMIT5: track 5.08 -> 367.3 mm, vias 0 -> 14
- net LIMIT3: track 5.13 -> 325.9 mm, vias 0 -> 10
- net LIMIT4: track 5.08 -> 270.6 mm, vias 0 -> 7
- net M0_STEP: track 260.9 -> 2.54 mm, vias 3 -> 0
- net M0_DIR: track 260.0 -> 2.54 mm, vias 4 -> 0
- net LIMIT2: track 5.08 -> 246.1 mm, vias 0 -> 10
- net M0_EN: track 236.9 -> 2.54 mm, vias 4 -> 0
- net LIMIT0: track 5.08 -> 230.3 mm, vias 0 -> 7
- net Net-(JP3-A): track 216.2 -> 0.00 mm, vias 3 -> 0
- net Net-(SW3-Pad1): track 25.0 -> 225.4 mm, vias 2 -> 3
- net Net-(SW4-Pad1): track 16.2 -> 215.3 mm, vias 0 -> 4
- net M2_EN: track 197.8 -> 0.00 mm, vias 2 -> 0
- net Net-(SW1-Pad1): track 46.7 -> 240.5 mm, vias 4 -> 3
- net LIMIT1: track 5.08 -> 198.0 mm, vias 0 -> 4
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Other:
- board text added: "3V3 Mega"
- board text added: "5V Mega"
- board text added: "5V Nano"
- board text added: "Designed by Parker, Rolston, et al"
- board text added: "Nano goes on bottom if installed."
- board text removed: "Designed by Parker and Rolston"

Commit message: Route nearly whole thing
Routing:
- net SDA: track 8.25 -> 358.8 mm, vias 0 -> 18
- net SCL: track 8.78 -> 344.8 mm, vias 0 -> 22
- net M0_STEP: track 2.54 -> 294.4 mm, vias 0 -> 7
- net M0_DIR: track 2.54 -> 288.1 mm, vias 0 -> 5
- net M0_EN: track 2.54 -> 276.5 mm, vias 0 -> 5
- net Net-(JP2-B): track 0.00 -> 182.6 mm, vias 0 -> 4
- net M5_STEP: track 0.00 -> 182.1 mm, vias 0 -> 3
- net M5_DIR: track 0.00 -> 175.2 mm, vias 0 -> 3
- net M5_EN: track 0.00 -> 159.9 mm, vias 0 -> 6
- net Net-(J5-Pin_3): track 2.54 -> 150.9 mm, vias 0 -> 6
- net Net-(J5-Pin_1): track 2.54 -> 147.8 mm, vias 0 -> 8
- net Net-(JP5-B): track 0.00 -> 135.8 mm, vias 0 -> 7
- net Net-(JP1-B): track 0.00 -> 133.0 mm, vias 0 -> 2
- net BUZZER0: track 0.00 -> 132.4 mm, vias 0 -> 6
- net M4_STEP: track 0.00 -> 129.2 mm, vias 0 -> 5
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