File: Arm_PCB/Arm_PCB.kicad_pcb (KiCad board)
At the start: 2 copper layers, 332.7 x 149.9 mm, 100 parts, among them J1 Conn_02x04_Counter_Clockwise, J10 Conn_02x02_Counter_Clockwise, J11 Conn_02x04_Counter_Clockwise, J12 Screw_Terminal_01x02, J13 Screw_Terminal_01x02, J14 Screw_Terminal_01x02, J15 Screw_Terminal_01x02, J16 Screw_Terminal_01x02, J17 Screw_Terminal_01x02, J18 Screw_Terminal_01x02, J19 Conn_02x03_Counter_Clockwise, J2 Conn_02x04_Counter_Clockwise, J20 Conn_02x03_Counter_Clockwise, J21 Screw_Terminal_01x02, J22 Screw_Terminal_01x02, J23 Screw_Terminal_01x02, J24 Screw_Terminal_01x02, J25 Screw_Terminal_01x02, J26 Screw_Terminal_01x02, J27 Screw_Terminal_01x02, J3 Conn_02x04_Counter_Clockwise, J4 Conn_02x04_Counter_Clockwise, J5 Conn_02x03_Counter_Clockwise, J6 Conn_02x07_Counter_Clockwise, J7 Conn_02x03_Counter_Clockwise, J8 Conn_02x02_Counter_Clockwise, J9 Conn_02x04_Counter_Clockwise, SW1 SW_Push, SW2 SW_Push, SW3 SW_Push, SW4 SW_Push, U1 TB6560_Board, U10 TB6560_Board, U11 INA219AxDCN, U12 TB6560_Board, U13 INA219AxDCN, U14 TB6560_Board, U15 INA219AxDCN, U16 TB6560_Board, U2 INA219AxDCN, U3 INA219AxDCN, U4 INA219AxDCN, U5 TB6560_Board, U6 INA219AxDCN, U7 TB6560_Board, U8 INA219AxDCN, U9 INA219AxDCN

Commit message: Finish PCB haha
Routing:
- net +5V: track 581.5 -> 592.7 mm
- net +24V: track 638.7 -> 634.9 mm
- net GND: vias 342 -> 382

Commit message: Add mounting holes, other minor changes
Parts:
- added H1: MountingHole, MountingHole:MountingHole_4.3mm_M4, F.Cu at (142.2, 91.4)
- added H2: MountingHole, MountingHole:MountingHole_4.3mm_M4, F.Cu at (368.3, 58.4)
- added H3: MountingHole, MountingHole:MountingHole_4.3mm_M4, F.Cu at (191.8, 47.0)
- added H4: MountingHole, MountingHole:MountingHole_4.3mm_M4, F.Cu at (293.4, 47.0)
- added H5: MountingHole, MountingHole:MountingHole_4.3mm_M4, F.Cu at (218.4, 92.7)
- added H6: MountingHole, MountingHole:MountingHole_4.3mm_M4, F.Cu at (330.2, 92.7)
- added H7: MountingHole, MountingHole:MountingHole_4.3mm_M4, F.Cu at (54.6, 182.9)
- added H8: MountingHole, MountingHole:MountingHole_4.3mm_M4, F.Cu at (90.2, 47.0)
- added H9: MountingHole, MountingHole:MountingHole_4.3mm_M4, F.Cu at (370.8, 186.7)
- moved J15 8.03 mm to (55.9, 172.7)
Routing:
- net +5V: track 592.7 -> 587.0 mm
