File: Arm_PCB/UXElements.kicad_sch (KiCad schematic)
At the start: 48 parts, among them J21 Screw_Terminal_01x02, J22 Screw_Terminal_01x02, J23 Screw_Terminal_01x02, J24 Screw_Terminal_01x02, J25 Screw_Terminal_01x02, J26 Screw_Terminal_01x02, J27 Screw_Terminal_01x02, J6 Conn_02x07_Counter_Clockwise

Commit message: Route more
Parts:
- removed D1, D2, D3, D4, D5, D6, D7: LED, LED_SMD:LED_1206_3216Metric_Pad1.42x1.75mm_HandSolder, symbol Device:LED
- removed R28, R29, R30, R31, R32, R33, R34: R, Resistor_SMD:R_1206_3216Metric_Pad1.30x1.75mm_HandSolder, symbol Device:R
Other:
- note removed: "Enable LEDs (EN is Active-Low, LEDs on when EN)"
